File: combined_board/EllieBoard.kicad_sch (KiCad schematic)
At the start: 13 parts, among them J1 Flow Meter Conn, J2 Servo Conn 1, J3 Servo Conn 2, J4 Dean Conn, U1 HX711, U2 HX711, U3 HX711, U4 HX711, U5 HX711, U6 HX711, U7 HX711, U8 HX711

Commit message: fixing some issues with schematic
Parts:
- removed U1, U2, U3, U4, U5, U6, U7, U8: HX711, symbol hx711:HX711
- added J10, J13, J14, J17, J18, J5, J6, J9: Conn_01x06_Male, symbol Connector:Conn_01x06_Male
- added J11, J12, J15, J16, J19, J20, J7, J8: Conn_01x04_Male, symbol Connector:Conn_01x04_Male
- added U?: HX711, symbol hx711:HX711
Connections:
- net +3V3: now also J10.6 (Pin_6), J13.6 (Pin_6), J14.6 (Pin_6), J17.6 (Pin_6), J18.6 (Pin_6), J5.6 (Pin_6), J6.6 (Pin_6), J9.6 (Pin_6)
- net GND: now also J11.3 (Pin_3), J11.4 (Pin_4), J12.3 (Pin_3), J12.4 (Pin_4), J15.3 (Pin_3), J15.4 (Pin_4), J16.3 (Pin_3), J16.4 (Pin_4), J19.3 (Pin_3), J19.4 (Pin_4), J20.3 (Pin_3), J20.4 (Pin_4), J7.3 (Pin_3), J7.4 (Pin_4), J8.3 (Pin_3), J8.4 (Pin_4)
- net IO12: now also J15.2 (Pin_2)
- net IO13: now also J19.2 (Pin_2)
- net IO14: now also J8.2 (Pin_2)
- net IO15: now also J12.2 (Pin_2)
- net IO16: now also J16.2 (Pin_2)
- net IO17: now also J20.2 (Pin_2)
- net IO4: now also J7.2 (Pin_2)
- net IO5: now also J11.2 (Pin_2)

Commit message: updated board electronics work session 04/04
Parts:
- removed J1: Flow Meter Conn, symbol Connector:Conn_01x03_Female
- removed J13, J14, J6: Conn_01x06_Male, symbol Connector:Conn_01x06_Male
- removed J15, J16, J8: Conn_01x04_Male, symbol Connector:Conn_01x04_Male
- removed U?: HX711, symbol hx711:HX711
- added J1: Load Cell 1.1, symbol Connector:Conn_01x04_Female
- added J13: Load Cell 4.1, symbol Connector:Conn_01x04_Female
- added J14: Load Cell 5.1, symbol Connector:Conn_01x04_Female
- added J15: Load Cell 6.1, symbol Connector:Conn_01x04_Female
- added J16, J24, J25: Conn_01x06_Male, symbol Connector:Conn_01x06_Male
- added J21, J26, J27: Conn_01x04_Male, symbol Connector:Conn_01x04_Male
- added J22: Load Cell 7.1, symbol Connector:Conn_01x04_Female
- added J23: Load Cell 8.1, symbol Connector:Conn_01x04_Female
- added J28: Flow Meter Conn 2, symbol Connector:Conn_01x03_Female
- added J29: Servo Conn 2, symbol Connector:Conn_01x03_Female
- added J30: Servo Conn 4, symbol Connector:Conn_01x03_Female
- added J31: Dean Conn 2, symbol Connector:Conn_01x02_Female
- added J32: Load Cell 1.2, symbol Connector:Conn_01x04_Female
- added J33: Load Cell 2.2, symbol Connector:Conn_01x04_Female
- added J34: Load Cell 3.2, symbol Connector:Conn_01x04_Female
- added J35: Load Cell 4.2, symbol Connector:Conn_01x04_Female
- added J36: Load Cell 5.2, symbol Connector:Conn_01x04_Female
- added J37: Load Cell 6.2, symbol Connector:Conn_01x04_Female
- added J38: Load Cell 7.2, symbol Connector:Conn_01x04_Female
- added J39: Load Cell 8.2, symbol Connector:Conn_01x04_Female
- added J40: SD Card Conn, symbol Connector:Conn_01x08_Male
- added J41: Flow Meter Conn 1, symbol Connector:Conn_01x03_Female
- added J42, J44: Relay Board Conn, symbol Connector:Conn_01x03_Female
- added J43: NC Conn, symbol Connector:Conn_01x02_Female
- added J6: Load Cell 2.1, symbol Connector:Conn_01x04_Female
- added J8: Load Cell 3.1, symbol Connector:Conn_01x04_Female
- added R1, R10, R12, R14, R16, R3, R5, R7: 820, Resistor_SMD:R_0201_0603Metric, symbol Device:R
- added R11, R13, R15, R17, R2, R4, R6, R8: 470, Resistor_SMD:R_0201_0603Metric, symbol Device:R
- added R9: 10k, Resistor_SMD:R_0201_0603Metric, symbol Device:R
- J3: value Servo Conn 2 -> Servo Conn 3
- J4: value Dean Conn -> Dean Conn 1
Connections:
- net +3V3: now also J11.4 (Pin_4), J12.4 (Pin_4), J19.4 (Pin_4), J20.4 (Pin_4), J7.4 (Pin_4), J16.6 (Pin_6), J21.4 (Pin_4), J24.6 (Pin_6), J25.6 (Pin_6), J26.4 (Pin_4), J27.4 (Pin_4), J40.8 (Pin_8), J42.1 (Pin_1), J44.2 (Pin_2), R1.2, R10.2, R12.2, R14.2, R16.2, R3.2, R5.2, R7.2
- net GND: now also J10.5 (Pin_5), J11.1 (Pin_1), J12.1 (Pin_1), J17.5 (Pin_5), J18.5 (Pin_5), J19.1 (Pin_1), J2.1 (Pin_1), J20.1 (Pin_1), J3.1 (Pin_1), J5.5 (Pin_5), J7.1 (Pin_1), J1.2 (Pin_2), J15.2 (Pin_2), J21.1 (Pin_1), J22.2 (Pin_2), J23.2 (Pin_2), J24.5 (Pin_5), J25.5 (Pin_5), J26.1 (Pin_1), J27.1 (Pin_1), J28.1 (Pin_1), J29.1 (Pin_1), J30.1 (Pin_1), J31.2 (Pin_2), J32.2 (Pin_2), J33.2 (Pin_2), J34.2 (Pin_2), J37.2 (Pin_2), J38.2 (Pin_2), J39.2 (Pin_2), J40.6 (Pin_6), J41.1 (Pin_1), J42.2 (Pin_2), J43.2 (Pin_2), J6.2 (Pin_2), J8.2 (Pin_2), R11.1, R13.1, R15.1, R17.1, R2.1, R4.1, R6.1, R8.1; no longer J11.3 (Pin_3), J11.4 (Pin_4), J12.3 (Pin_3), J12.4 (Pin_4), J19.3 (Pin_3), J19.4 (Pin_4), J2.3 (Pin_3), J20.3 (Pin_3), J20.4 (Pin_4), J3.3 (Pin_3), J7.3 (Pin_3), J7.4 (Pin_4)
- net IO12: now also J27.3 (Pin_3)
- net IO13: now also J26.3 (Pin_3); no longer J19.2 (Pin_2)
- net IO14: now also J11.3 (Pin_3)
- net IO15: now also J19.3 (Pin_3); no longer J12.2 (Pin_2)
- net IO16: now also J12.3 (Pin_3)
- net IO17: now also J20.3 (Pin_3); no longer J20.2 (Pin_2)
- net IO18: now also J7.2 (Pin_2), J28.2 (Pin_2), J41.2 (Pin_2)
- net IO19: now also J2.2 (Pin_2), J21.2 (Pin_2), J29.2 (Pin_2); no longer J2.1 (Pin_1)
- net IO21: now also J3.2 (Pin_2), J27.2 (Pin_2), J30.2 (Pin_2); no longer J3.1 (Pin_1)
- net IO4: now also J7.3 (Pin_3); no longer J7.2 (Pin_2)
- net IO5: now also J21.3 (Pin_3); no longer J11.2 (Pin_2)
- net A2-: now reaches J18.3 (Pin_3)
- net A2-: now also J33.4 (Pin_4), J6.4 (Pin_4)
- net A2+: now reaches J18.4 (Pin_4)
- net A2+: now also J33.3 (Pin_3), J6.3 (Pin_3)
- net A8-: now reaches J17.3 (Pin_3)
- net A8-: now also J23.4 (Pin_4)
- net A8+: now reaches J17.4 (Pin_4)
- net A8+: now also J23.3 (Pin_3), J39.3 (Pin_3)
- net IO25: now reaches MOD1.10 (IO25)
- net IO25: now also J19.2 (Pin_2)
- net IO26: now reaches MOD1.11 (IO26)
- net IO26: now also J12.2 (Pin_2)
- net IO27: now reaches MOD1.12 (IO27)
- net IO27: now also J20.2 (Pin_2)
- net SCK/CLK: now reaches MOD1.20 (SCK/CLK)
- net SCK/CLK: now also J40.5 (Pin_5)
- net SDO/SD0: now reaches MOD1.21 (SDO/SD0)
- net SDO/SD0: now also J40.4 (Pin_4)
- net SDI/SD1: now reaches MOD1.22 (SDI/SD1)
- net SDI/SD1: now also J40.3 (Pin_3)
- net IO2: now reaches MOD1.24 (IO2)
- net IO2: now also J40.2 (Pin_2)
- net IO22: now reaches MOD1.36 (IO22)
- net IO22: now also J26.2 (Pin_2)
- net IO23: now reaches MOD1.37 (IO23)
- net IO23: now also J11.2 (Pin_2)
- net IO34: now reaches MOD1.6 (IO34)
- net IO34: now also MOD1.9 (IO33), R9.1
- net IO35: now reaches MOD1.7 (IO35)
- net IO35: now also J42.3 (Pin_3)
- net IO32: now reaches MOD1.8 (IO32)
- net A7-: now reaches J10.3 (Pin_3)
- net A7-: now also J22.4 (Pin_4), J38.4 (Pin_4)
- net A7+: now reaches J10.4 (Pin_4)
- net A7+: now also J22.3 (Pin_3), J38.3 (Pin_3)
- net A4-: now reaches J9.3 (Pin_3)
- net A4-: now also J13.4 (Pin_4), J35.4 (Pin_4)
- net A4+: now reaches J9.4 (Pin_4)
- net A4+: now also J13.3 (Pin_3), J35.3 (Pin_3)
- net A1-: now reaches J5.3 (Pin_3)
- net A1-: now also J1.4 (Pin_4), J32.4 (Pin_4)
- net A1+: now reaches J5.4 (Pin_4)
- net A1+: now also J1.3 (Pin_3), J32.3 (Pin_3)
- removed net Lipo 5V: J2.2 (Pin_2), J3.2 (Pin_2), J4.1 (Pin_1)
- new net: R3.1, R4.2
- new net: J40.1 (Pin_1), R9.2
- new net A3+: J25.4 (Pin_4), J34.3 (Pin_3), J8.3 (Pin_3)
- new net A3-: J25.3 (Pin_3), J34.4 (Pin_4), J8.4 (Pin_4)
- new net A5+: J14.3 (Pin_3), J16.4 (Pin_4), J36.3 (Pin_3)
- new net A5-: J14.4 (Pin_4), J16.3 (Pin_3), J36.4 (Pin_4)
- new net A6+: J15.3 (Pin_3), J24.4 (Pin_4), J37.3 (Pin_3)
- new net A6-: J15.4 (Pin_4), J24.3 (Pin_3), J37.4 (Pin_4)
- new net Lipo: J2.3 (Pin_3), J29.3 (Pin_3), J3.3 (Pin_3), J30.3 (Pin_3), J4.1 (Pin_1), J41.3 (Pin_3)
- new net Lipo : J28.3 (Pin_3), J31.1 (Pin_1)
- new net NC: J43.1 (Pin_1), J44.3 (Pin_3)
- new net out1: J1.1 (Pin_1), J32.1 (Pin_1), R1.1, R2.2
- new net out2: J33.1 (Pin_1), J6.1 (Pin_1), R10.1, R13.2
- new net out3: J34.1 (Pin_1), J8.1 (Pin_1), R16.1, R17.2
- new net out4: J13.1 (Pin_1), J35.1 (Pin_1)
- new net out5: J14.1 (Pin_1), J36.1 (Pin_1), R7.1, R8.2
- new net out6: J15.1 (Pin_1), J37.1 (Pin_1), R14.1, R15.2
- new net out7: J22.1 (Pin_1), J38.1 (Pin_1), R5.1, R6.2
- new net out8: J23.1 (Pin_1), J39.1 (Pin_1), R11.2, R12.1
- new net u4: J13.2 (Pin_2), J35.2 (Pin_2)
- new net u5: J14.2 (Pin_2), J16.5 (Pin_5), J36.2 (Pin_2)
Other:
- moved on the sheet: J2, J3, J4, J5, J7, MOD1

Commit message: kicad board work
custom board updates
Parts:
- removed J10, J16, J17, J18, J24, J25, J5, J9: Conn_01x06_Male, symbol Connector:Conn_01x06_Male
- removed J11, J12, J19, J20, J21, J26, J27, J7: Conn_01x04_Male, symbol Connector:Conn_01x04_Male
- removed J31: Dean Conn 2, symbol Connector:Conn_01x02_Female
- removed J40: SD Card Conn, symbol Connector:Conn_01x08_Male
- removed J42, J44: Relay Board Conn, symbol Connector:Conn_01x03_Female
- removed MOD1: ESP32-WROOM-32, digikey-footprints:ESP32-WROOM-32D, symbol dk_RF-Transceiver-Modules:ESP32-WROOM-32
- added J5, J7: NC Conn 2, TerminalBlock_Phoenix:TerminalBlock_Phoenix_MPT-0,5-2-2.54_1x02_P2.54mm_Horizontal, symbol Connector:Conn_01x02_Female
- added U1, U10, U11, U2, U5, U6, U8, U9: HX711_Breakout, Ellie_Project_Footprints:HX711_Breakout_Board, symbol ELLIE_Symbol_Library:HX711_Breakout
- added U3: Relay_Board, Ellie_Project_Footprints:Relay_Breakout, symbol ELLIE_Symbol_Library:Relay_Board
- added U4: SD_Card_Reader, Ellie_Project_Footprints:SD_Card_Breakout, symbol ELLIE_Symbol_Library:SD_Card_Reader
- added U7: ESP32-DEVKITC-32D, ESP32-DEVKITC-32D:MODULE_ESP32-DEVKITC-32D, symbol ESP32-DEVKITC-32D:ESP32-DEVKITC-32D
- J1, J13, J14, J15, J22, J23, J6, J8: footprint (none) -> Connector_JST:JST_XH_B4B-XH-AM_1x04_P2.50mm_Vertical
- J2, J3, J41: footprint (none) -> Connector_JST:JST_XH_B3B-XH-AM_1x03_P2.50mm_Vertical
- J28, J29, J30: footprint (none) -> TerminalBlock_Phoenix:TerminalBlock_Phoenix_MPT-0,5-3-2.54_1x03_P2.54mm_Horizontal
- J32, J33, J34, J35, J36, J37, J38, J39: footprint (none) -> TerminalBlock_Phoenix:TerminalBlock_Phoenix_MPT-0,5-4-2.54_1x04_P2.54mm_Horizontal
- J4: value Dean Conn 1 -> NC Conn; footprint (none) -> Connector_JST:JST_XH_B2B-XH-AM_1x02_P2.50mm_Vertical
- J43: footprint (none) -> Connector_JST:JST_XH_B2B-XH-AM_1x02_P2.50mm_Vertical
- R1, R10, R11, R12, R13, R14, R15, R16, R17, R2, R3, R4, R5, R6, R7, R8, R9: footprint Resistor_SMD:R_0201_0603Metric -> Resistor_SMD:R_1206_3216Metric
Connections:
- net Lipo  is gone; now on net GND: J28.3 (Pin_3)
- net NC is gone; now on net Lipo: J43.1 (Pin_1)
- net +3V3: now also R9.1, U1.10 (VCC), U10.10 (VCC), U11.10 (VCC), U2.10 (VCC), U4.7 (3V), U5.10 (VCC), U6.10 (VCC), U7.1 (3V3), U8.10 (VCC), U9.10 (VCC); no longer R1.2, R10.2, R12.2, R14.2, R16.2, R3.2, R5.2, R7.2
- net A1+: now also J1.4 (Pin_4), J32.4 (Pin_4), U1.4 (A+); no longer J1.3 (Pin_3), J32.3 (Pin_3)
- net A1-: now also J1.3 (Pin_3), J32.3 (Pin_3), U1.3 (A-); no longer J1.4 (Pin_4), J32.4 (Pin_4)
- net A2+: now also J33.4 (Pin_4), J6.4 (Pin_4), U6.4 (A+); no longer J33.3 (Pin_3), J6.3 (Pin_3)
- net A2-: now also J33.3 (Pin_3), J6.3 (Pin_3), U6.3 (A-); no longer J33.4 (Pin_4), J6.4 (Pin_4)
- net A3+: now also J34.4 (Pin_4), J8.4 (Pin_4), U8.4 (A+); no longer J34.3 (Pin_3), J8.3 (Pin_3)
- net A3-: now also J34.3 (Pin_3), J8.3 (Pin_3), U8.3 (A-); no longer J34.4 (Pin_4), J8.4 (Pin_4)
- net A4+: now also J13.4 (Pin_4), J35.4 (Pin_4), U11.4 (A+); no longer J13.3 (Pin_3), J35.3 (Pin_3)
- net A4-: now also J13.3 (Pin_3), J35.3 (Pin_3), U11.3 (A-); no longer J13.4 (Pin_4), J35.4 (Pin_4)
- net A5+: now also J14.4 (Pin_4), J36.4 (Pin_4), U2.4 (A+); no longer J14.3 (Pin_3), J36.3 (Pin_3)
- net A5-: now also J14.3 (Pin_3), J36.3 (Pin_3), U2.3 (A-); no longer J14.4 (Pin_4), J36.4 (Pin_4)
- net A6+: now also J15.4 (Pin_4), J37.4 (Pin_4), U5.4 (A+); no longer J15.3 (Pin_3), J37.3 (Pin_3)
- net A6-: now also J15.3 (Pin_3), J37.3 (Pin_3), U5.3 (A-); no longer J15.4 (Pin_4), J37.4 (Pin_4)
- net A7+: now also J22.4 (Pin_4), J38.4 (Pin_4), U9.4 (A+); no longer J22.3 (Pin_3), J38.3 (Pin_3)
- net A7-: now also J22.3 (Pin_3), J38.3 (Pin_3), U9.3 (A-); no longer J22.4 (Pin_4), J38.4 (Pin_4)
- net A8+: now also J23.4 (Pin_4), J39.4 (Pin_4), U10.4 (A+); no longer J23.3 (Pin_3), J39.3 (Pin_3)
- net A8-: now also J23.3 (Pin_3), J39.3 (Pin_3), U10.3 (A-); no longer J23.4 (Pin_4)
- net GND: now also J2.3 (Pin_3), J29.3 (Pin_3), J3.3 (Pin_3), J30.3 (Pin_3), J41.3 (Pin_3), J5.2 (Pin_2), J7.2 (Pin_2), U1.7 (GND), U10.7 (GND), U11.7 (GND), U2.7 (GND), U3.4 (GND), U4.6 (GND), U5.7 (GND), U6.7 (GND), U7.14 (GND1), U7.20 (GND3), U7.26 (GND2), U8.7 (GND), U9.7 (GND); no longer J1.2 (Pin_2), J15.2 (Pin_2), J2.1 (Pin_1), J22.2 (Pin_2), J23.2 (Pin_2), J28.1 (Pin_1), J29.1 (Pin_1), J3.1 (Pin_1), J30.1 (Pin_1), J32.2 (Pin_2), J33.2 (Pin_2), J34.2 (Pin_2), J37.2 (Pin_2), J38.2 (Pin_2), J39.2 (Pin_2), J41.1 (Pin_1), J6.2 (Pin_2), J8.2 (Pin_2)
- net IO12: now also J2.2 (Pin_2), J29.2 (Pin_2), U7.13 (IO12)
- net IO13: now also J3.2 (Pin_2), J30.2 (Pin_2), U7.15 (IO13)
- net IO14: now also U3.3 (IN2), U7.12 (IO14)
- net IO15: now also U6.8 (DT), U7.35 (IO15)
- net IO16: now also R9.2, U4.1 (CD), U7.31 (IO16)
- net IO17: now also U4.2 (CS), U7.30 (IO17)
- net IO18: now also U7.28 (IO18)
- net IO19: now also U11.8 (DT), U7.27 (IO19); no longer J2.2 (Pin_2), J29.2 (Pin_2)
- net IO2: now also U6.9 (SCK), U7.34 (IO2)
- net IO21: now also U11.9 (SCK), U7.25 (IO21); no longer J3.2 (Pin_2), J30.2 (Pin_2)
- net IO22: now also U7.22 (IO22), U8.8 (DT)
- net IO23: now also U7.21 (IO23), U8.9 (SCK)
- net IO25: now also U2.9 (SCK), U7.9 (IO25)
- net IO26: now also U5.9 (SCK), U7.10 (IO26)
- net IO27: now also U3.2 (IN1), U7.11 (IO27)
- net IO32: now also U1.8 (DT), U10.9 (SCK), U7.32 (IO4), U7.7 (IO32)
- net IO34: now also U5.8 (DT), U7.5 (IO34); no longer R9.1
- net IO35: now also U2.8 (DT), U7.6 (IO35)
- net IO5: now also U1.9 (SCK), U7.29 (IO5)
- net Lipo: now also J2.1 (Pin_1), J29.1 (Pin_1), J3.1 (Pin_1), J30.1 (Pin_1), J5.1 (Pin_1), J7.1 (Pin_1); no longer J2.3 (Pin_3), J29.3 (Pin_3), J3.3 (Pin_3), J30.3 (Pin_3), J41.3 (Pin_3)
- net SCK/CLK: now also U4.5 (CK), U7.23 (TXD0)
- net SDI/SD1: now also U4.3 (DI), U7.33 (IO0)
- net SDO/SD0: now also U4.4 (DO), U7.24 (RXD0)
- net out4: now also R3.1, R4.2
- net u4: now also U11.2 (E-)
- net u5: now also U2.2 (E-)
- new net: R3.2, U11.1 (E+)
- new net: R10.2, U6.1 (E+)
- new net: R7.2, U2.1 (E+)
- new net: R5.2, U9.1 (E+)
- new net: R12.2, U10.1 (E+)
- new net: R14.2, U5.1 (E+)
- new net: R16.2, U8.1 (E+)
- new net: R1.2, U1.1 (E+)
- new net +5V: J28.1 (Pin_1), J41.1 (Pin_1), U3.1 (VCC), U7.19 (EXT_5V)
- new net IO33: U7.8 (IO33), U9.9 (SCK)
- new net IO36: U10.8 (DT), U7.3 (SENSOR_VP)
- new net IO39: U7.4 (SENSOR_VN), U9.8 (DT)
- new net u1: J1.2 (Pin_2), J32.2 (Pin_2), U1.2 (E-)
- new net u2: J33.2 (Pin_2), J6.2 (Pin_2), U6.2 (E-)
- new net u3: J34.2 (Pin_2), J8.2 (Pin_2), U8.2 (E-)
- new net u6: J15.2 (Pin_2), J37.2 (Pin_2), U5.2 (E-)
- new net u7: J22.2 (Pin_2), J38.2 (Pin_2), U9.2 (E-)
- new net u8: J23.2 (Pin_2), J39.2 (Pin_2), U10.2 (E-)
- no-connect marks 0 -> 24
Other:
- moved on the sheet: J43, R9

Commit message: Layout updates 04/05
Parts:
- added J9: Battery Conn, Connector_JST:JST_XH_B2B-XH-AM_1x02_P2.50mm_Vertical, symbol Connector:Conn_01x02_Female
Connections:
- net GND: now also J9.2 (Pin_2)
- net Lipo: now also J9.1 (Pin_1)
Changed lines of the file:
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@@
     (stroke (width 0) (type default) (color 0 0 0 0))
   )
+  (wire (pts (xy 132.08 166.37) (xy 137.16 166.37))
+    (stroke (width 0) (type default) (color 0 0 0 0))
+  )
   (wire (pts (xy 129.54 125.73) (xy 133.35 125.73))
     (stroke (width 0) (type default) (color 0 0 0 0))
@@
     (stroke (width 0) (type default) (color 0 0 0 0))
   )
+  (wire (pts (xy 134.62 163.83) (xy 137.16 163.83))
+    (stroke (width 0) (type default) (color 0 0 0 0))
+  )
   (wire (pts (xy 133.35 115.57) (xy 129.54 115.57))
     (stroke (width 0) (type default) (color 0 0 0 0))
@@
     )
   )
+  (global_label "Lipo" (shape input) (at 134.62 163.83 180) (fields_autoplaced)
+    (effects (font (size 1.27 1.27)) (justify right))
+    (property "Intersheet References" "${INTERSHEET_REFS}" (id 0) (at 128.2759 163.7506 0)
+      (effects (font (size 1.27 1.27)) (justify right) hide)
+    )
+  )
   (global_label "out5" (shape input) (at 43.18 146.05 180) (fields_autoplaced)
     (effects (font (size 1.27 1.27)) (justify right))
@@
     (pin "1")
   )
+  (symbol (lib_id "Connector:Conn_01x02_Female") (at 142.24 163.83 0) (unit 1)
+    (in_bom yes) (on_board yes)
+    (property "Reference" "J9" (id 0) (at 143.51 163.8299 0)
+      (effects (font (size 1.27 1.27)) (justify left))
+    )
+    (property "Value" "Battery Conn" (id 1) (at 147.32 170.18 90)
+      (effects (font (size 1.27 1.27)) (justify left))
+    )
+    (property "Footprint" "Connector_JST:JST_XH_B2B-XH-AM_1x02_P2.50mm_Vertical" (id 2) (at 142.24 163.83 0)
+      (effects (font (size 1.27 1.27)) hide)
+    )
+    (property "Datasheet" "~" (id 3) (at 142.24 163.83 0)
+      (effects (font (size 1.27 1.27)) hide)
+    )
+    (pin "1")
+    (pin "2")
+  )
   (symbol (lib_id "power:GND") (at 104.14 119.38 0) (unit 1)
     (in_bom yes) (on_board yes) (fields_autoplaced)
@@
     (pin "8")
   )
+  (symbol (lib_id "power:GND") (at 132.08 166.37 0) (unit 1)
+    (in_bom yes) (on_board yes) (fields_autoplaced)
+    (property "Reference" "#PWR0112" (id 0) (at 132.08 172.72 0)
+      (effects (font (size 1.27 1.27)) hide)
+    )
+    (property "Value" "GND" (id 1) (at 132.08 171.45 0))
+    (property "Footprint" "" (id 2) (at 132.08 166.37 0)
+      (effects (font (size 1.27 1.27)) hide)
+    )
+    (property "Datasheet" "" (id 3) (at 132.08 166.37 0)
+      (effects (font (size 1.27 1.27)) hide)
+    )
+    (pin "1")
+  )
   (symbol (lib_id "power:GND") (at 21.59 78.74 0) (unit 1)
     (in_bom yes) (on_board yes) (fields_autoplaced)
@@
       (reference "#PWR0111") (unit 1) (value "GND") (footprint "")
     )
+    (path "/eb5c933c-98d8-4a80-8f61-a13118588388"
+      (reference "#PWR0112") (unit 1) (value "GND") (footprint "")
+    )
     (path "/371c524c-8f82-45c2-afb1-cab047f19c98"
       (reference "J1") (unit 1) (value "Load Cell 1.1") (footprint "Connector_JST:JST_XH_B4B-XH-AM_1x04_P2.50mm_Vertical")
@@
       (reference "J8") (unit 1) (value "Load Cell 3.1") (footprint "Connector_JST:JST_XH_B4B-XH-AM_1x04_P2.50mm_Vertical")
     )
+    (path "/88f181e9-e191-43c6-b7be-c4c3e06c0ee7"
+      (reference "J9") (unit 1) (value "Battery Conn") (footprint "Connector_JST:JST_XH_B2B-XH-AM_1x02_P2.50mm_Vertical")
+    )
     (path "/957106c1-c369-479a-bc59-780f64836b56"
