File: combined_board/EllieBoard.kicad_sch (KiCad schematic)
At the start: 55 parts, among them J1 Load Cell 1.1, J13 Load Cell 4.1, J14 Load Cell 5.1, J15 Load Cell 6.1, J2 Servo Conn 1, J22 Load Cell 7.1, J23 Load Cell 8.1, J28 Flow Meter Conn 2, J29 Servo Conn 2, J3 Servo Conn 3, J30 Servo Conn 4, J32 Load Cell 1.2, J33 Load Cell 2.2, J34 Load Cell 3.2, J35 Load Cell 4.2, J36 Load Cell 5.2, J37 Load Cell 6.2, J38 Load Cell 7.2, J39 Load Cell 8.2, J4 NC Conn, J41 Flow Meter Conn 1, J43 NC Conn, J5 NC Conn 2, J6 Load Cell 2.1, J7 NC Conn 2, J8 Load Cell 3.1, J9 Battery Conn, U1 HX711_Breakout, U10 HX711_Breakout, U11 HX711_Breakout, U2 HX711_Breakout, U3 Relay_Board, U4 SD_Card_Reader, U5 HX711_Breakout, U6 HX711_Breakout, U7 ESP32-DEVKITC-32D, U8 HX711_Breakout, U9 HX711_Breakout

Commit message: Kicad board connector and silkscreen fixes
Parts:
- added J10: Battery Conn Backup, Connector_JST:JST_XH_B2B-XH-AM_1x02_P2.50mm_Vertical, symbol Connector:Conn_01x02_Female
- added J11: Battery Conn Backup 2, TerminalBlock_Phoenix:TerminalBlock_Phoenix_MPT-0,5-2-2.54_1x02_P2.54mm_Horizontal, symbol Connector:Conn_01x02_Female
- J9: footprint Connector_JST:JST_XH_B2B-XH-AM_1x02_P2.50mm_Vertical -> Ellie_Project_Footprints:DEANS
Connections:
- net GND: now also J10.2 (Pin_2), J11.2 (Pin_2)
- net Lipo: now also J10.1 (Pin_1), J11.1 (Pin_1)
Changed lines of the file:
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@@
     (stroke (width 0) (type default) (color 0 0 0 0))
   )
+  (wire (pts (xy 156.21 182.88) (xy 161.29 182.88))
+    (stroke (width 0) (type default) (color 0 0 0 0))
+  )
   (wire (pts (xy 227.33 63.5) (xy 229.87 63.5))
     (stroke (width 0) (type default) (color 0 0 0 0))
@@
     (stroke (width 0) (type default) (color 0 0 0 0))
   )
+  (wire (pts (xy 158.75 180.34) (xy 161.29 180.34))
+    (stroke (width 0) (type default) (color 0 0 0 0))
+  )
   (wire (pts (xy 125.73 27.94) (xy 125.73 33.02))
     (stroke (width 0) (type default) (color 0 0 0 0))
@@
     (stroke (width 0) (type default) (color 0 0 0 0))
   )
+  (wire (pts (xy 132.08 182.88) (xy 137.16 182.88))
+    (stroke (width 0) (type default) (color 0 0 0 0))
+  )
   (wire (pts (xy 41.91 90.17) (xy 43.18 90.17))
     (stroke (width 0) (type default) (color 0 0 0 0))
@@
     (stroke (width 0) (type default) (color 0 0 0 0))
   )
+  (wire (pts (xy 134.62 180.34) (xy 137.16 180.34))
+    (stroke (width 0) (type default) (color 0 0 0 0))
+  )
   (wire (pts (xy 133.35 115.57) (xy 129.54 115.57))
     (stroke (width 0) (type default) (color 0 0 0 0))
@@
     )
   )
+  (global_label "Lipo" (shape input) (at 134.62 180.34 180) (fields_autoplaced)
+    (effects (font (size 1.27 1.27)) (justify right))
+    (property "Intersheet References" "${INTERSHEET_REFS}" (id 0) (at 128.2759 180.2606 0)
+      (effects (font (size 1.27 1.27)) (justify right) hide)
+    )
+  )
   (global_label "A2+" (shape input) (at 43.18 111.76 180) (fields_autoplaced)
     (effects (font (size 1.27 1.27)) (justify right))
@@
     )
   )
+  (global_label "Lipo" (shape input) (at 158.75 180.34 180) (fields_autoplaced)
+    (effects (font (size 1.27 1.27)) (justify right))
+    (property "Intersheet References" "${INTERSHEET_REFS}" (id 0) (at 152.4059 180.2606 0)
+      (effects (font (size 1.27 1.27)) (justify right) hide)
+    )
+  )
   (global_label "IO34" (shape input) (at 129.54 113.03 180) (fields_autoplaced)
     (effects (font (size 1.27 1.27)) (justify right))
@@
     (pin "1")
   )
+  (symbol (lib_id "Connector:Conn_01x02_Female") (at 166.37 180.34 0) (unit 1)
+    (in_bom yes) (on_board yes)
+    (property "Reference" "J11" (id 0) (at 167.64 180.3399 0)
+      (effects (font (size 1.27 1.27)) (justify left))
+    )
+    (property "Value" "Battery Conn Backup 2" (id 1) (at 171.45 191.77 90)
+      (effects (font (size 1.27 1.27)) (justify left))
+    )
+    (property "Footprint" "TerminalBlock_Phoenix:TerminalBlock_Phoenix_MPT-0,5-2-2.54_1x02_P2.54mm_Horizontal" (id 2) (at 166.37 180.34 0)
+      (effects (font (size 1.27 1.27)) hide)
+    )
+    (property "Datasheet" "~" (id 3) (at 166.37 180.34 0)
+      (effects (font (size 1.27 1.27)) hide)
+    )
+    (pin "1")
+    (pin "2")
+  )
   (symbol (lib_id "power:GND") (at 261.62 29.21 0) (unit 1)
     (in_bom yes) (on_board yes) (fields_autoplaced)
@@
     (pin "2")
   )
+  (symbol (lib_id "power:GND") (at 132.08 182.88 0) (unit 1)
+    (in_bom yes) (on_board yes) (fields_autoplaced)
+    (property "Reference" "#PWR0114" (id 0) (at 132.08 189.23 0)
+      (effects (font (size 1.27 1.27)) hide)
+    )
+    (property "Value" "GND" (id 1) (at 132.08 187.96 0))
+    (property "Footprint" "" (id 2) (at 132.08 182.88 0)
+      (effects (font (size 1.27 1.27)) hide)
+    )
+    (property "Datasheet" "" (id 3) (at 132.08 182.88 0)
+      (effects (font (size 1.27 1.27)) hide)
+    )
+    (pin "1")
+  )
   (symbol (lib_id "power:GND") (at 212.09 111.76 0) (unit 1)
     (in_bom yes) (on_board yes) (fields_autoplaced)
@@
     (pin "1")
   )
+  (symbol (lib_id "power:GND") (at 156.21 182.88 0) (unit 1)
+    (in_bom yes) (on_board yes) (fields_autoplaced)
+    (property "Reference" "#PWR0113" (id 0) (at 156.21 189.23 0)
+      (effects (font (size 1.27 1.27)) hide)
+    )
+    (property "Value" "GND" (id 1) (at 156.21 187.96 0))
+    (property "Footprint" "" (id 2) (at 156.21 182.88 0)
+      (effects (font (size 1.27 1.27)) hide)
+    )
+    (property "Datasheet" "" (id 3) (at 156.21 182.88 0)
+      (effects (font (size 1.27 1.27)) hide)
+    )
+    (pin "1")
+  )
   (symbol (lib_id "power:GND") (at 107.95 190.5 0) (unit 1)
     (in_bom yes) (on_board yes) (fields_autoplaced)
@@
       (effects (font (size 1.27 1.27)) (justify left))
     )
-    (property "Footprint" "Connector_JST:JST_XH_B2B-XH-AM_1x02_P2.50mm_Vertical" (id 2) (at 142.24 163.83 0)
+    (property "Footprint" "Ellie_Project_Footprints:DEANS" (id 2) (at 142.24 163.83 0)
       (effects (font (size 1.27 1.27)) hide)
     )
@@
     (pin "2")
   )
+  (symbol (lib_id "Connector:Conn_01x02_Female") (at 142.24 180.34 0) (unit 1)
+    (in_bom yes) (on_board yes)
+    (property "Reference" "J10" (id 0) (at 143.51 180.3399 0)
+      (effects (font (size 1.27 1.27)) (justify left))
+    )
+    (property "Value" "Battery Conn Backup" (id 1) (at 147.32 191.77 90)
+      (effects (font (size 1.27 1.27)) (justify left))
+    )
+    (property "Footprint" "Connector_JST:JST_XH_B2B-XH-AM_1x02_P2.50mm_Vertical" (id 2) (at 142.24 180.34 0)
+      (effects (font (size 1.27 1.27)) hide)
+    )
+    (property "Datasheet" "~" (id 3) (at 142.24 180.34 0)
+      (effects (font (size 1.27 1.27)) hide)
+    )
+    (pin "1")
+    (pin "2")
+  )
   (symbol (lib_id "Connector:Conn_01x04_Female") (at 27.94 120.65 0) (unit 1)
     (in_bom yes) (on_board yes)
@@
       (reference "#PWR0112") (unit 1) (value "GND") (footprint "")
     )
+    (path "/439e6463-0296-4527-8dc6-47fb96e37143"
+      (reference "#PWR0113") (unit 1) (value "GND") (footprint "")
+    )
+    (path "/28d95701-1ce4-4407-9f61-1674332e1642"
+      (reference "#PWR0114") (unit 1) (value "GND") (footprint "")
+    )
     (path "/371c524c-8f82-45c2-afb1-cab047f19c98"
       (reference "J1") (unit 1) (value "Load Cell 1.1") (footprint "Connector_JST:JST_XH_B4B-XH-AM_1x04_P2.50mm_Vertical")
@@
     )
     (path "/88f181e9-e191-43c6-b7be-c4c3e06c0ee7"
-      (reference "J9") (unit 1) (value "Battery Conn") (footprint "Connector_JST:JST_XH_B2B-XH-AM_1x02_P2.50mm_Vertical")
+      (reference "J9") (unit 1) (value "Battery Conn") (footprint "Ellie_Project_Footprints:DEANS")
+    )
+    (path "/d2a2d595-c71b-425e-a2be-8543c0300d91"
+      (reference "J10") (unit 1) (value "Battery Conn Backup") (footprint "Connector_JST:JST_XH_B2B-XH-AM_1x02_P2.50mm_Vertical")
+    )
+    (path "/111c38f7-ec2b-444f-8ec0-61814dc6a219"
+      (reference "J11") (unit 1) (value "Battery Conn Backup 2") (footprint "TerminalBlock_Phoenix:TerminalBlock_Phoenix_MPT-0,5-2-2.54_1x02_P2.54mm_Horizontal")
     )
     (path "/957106c1-c369-479a-bc59-780f64836b56"
